File: hardware/reflow-controller/reflow-controller.kicad_pcb (KiCad board)
At the start: 2 copper layers, 96.5 x 47.5 mm, 89 parts, among them J1 Conn_01x04, J10 BOOT_SEL, J2 Conn_01x04, J3 2.54mm Header, J4 ADC, J5 Conn_02x07_Odd_Even, J6 USB_B, J7 5.08mm Screw Terminal, J8 5.08mm Screw Terminal, J9 5.08mm Screw Terminal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

Commit message: Fixed error with shorting 5V and GND
Routing:
- net GND: vias 41 -> 40
Changed lines of the file:
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@@
     (thickness 1.6)
     (drawings 6)
-    (tracks 619)
+    (tracks 618)
     (zones 0)
     (modules 89)
@@
   (via (at 128.7 141.6) (size 0.8) (drill 0.4) (layers F.Cu B.Cu) (net 1))
   (via (at 136.7 141.2) (size 0.8) (drill 0.4) (layers F.Cu B.Cu) (net 1))
-  (via (at 129.7 132.1) (size 0.8) (drill 0.4) (layers F.Cu B.Cu) (net 1))
   (segment (start 136.8135 131.0865) (end 136.8135 132.4135) (width 1) (layer F.Cu) (net 1))
   (via (at 136.8135 131.0865) (size 0.8) (drill 0.4) (layers F.Cu B.Cu) (net 1))
@@
   (segment (start 167 110.5) (end 165.824999 109.324999) (width 0.25) (layer F.Cu) (net 95))
   (zone (net 6) (net_name +5V) (layer F.Cu) (hatch edge 0.508)
+    (priority 1)
     (connect_pads (clearance 0.508))
     (min_thickness 0.254)
